File: LarryLabFunctionGen.kicad_sch (KiCad schematic)
At the start: 0 parts

Commit message: added pulse gen and other stuff
Parts:
- added R7: 10k, symbol Device:R_US
- added V1, V2: 15, symbol Simulation_SPICE:VDC
- added V3: 2.0, symbol Simulation_SPICE:VDC
Connections:
- new net +15V: V1.1
- new net -15V: V2.2
- new net GND: R7.2, V1.2, V2.1, V3.2
- new net Larry Oscillator/GATE: R7.1, V3.1
Other:
- added sheet Pulse Generator (pulse_gen.kicad_sch)
- sheet Larry Oscillator ports: added GATE; removed none
- sheet Ouput Stage ports: added PULSE; removed none

Commit message: post wed changes
Other:
- sheet Pulse Generator ports: added none; removed GATE
Changed lines of the file:
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@@
-	)
-	(junction
-		(at 55.88 121.92)
-		(diameter 0)
-		(color 0 0 0 0)
 	)
 	(junction
@@
 		(pts
 			(xy 43.18 85.09) (xy 53.34 85.09)
-		)
-		(stroke
-			(width 0)
-			(type default)
-		)
-	)
-	(wire
-		(pts
-			(xy 124.46 121.92) (xy 55.88 121.92)
 		)
 		(stroke
@@
 			)
 		)
-		(pin "GATE" input
-			(at 124.46 121.92 180)
-			(effects
-				(font
-					(size 1.27 1.27)
-				)
-				(justify left)
-			)
-		)
